File: BMS.kicad_sch (KiCad schematic)
At the start: 112 parts, among them J1 USB_C_Receptacle_USB2.0_16P, J2 Conn_01x02_Pin, J3 Conn_01x02_Pin, J4 Conn_01x05_Pin, J5 Conn_01x02_Pin, J6 Conn_01x04_Pin, Q1 MMFTP3401-AQ, Q3 SS8050, Q4 IRLZ44N, Q5 IRLZ44N, Q6 IRLZ44N, Q7 IRF4905, Q8 IRF4905, Q9 SS8050, SW1 SW_MEC_5G, SW2 SW_MEC_5G, U1 USBLC6-2SC6, U11 INA213AIDCKT, U12 SFH617A-3X007T, U13 SFH617A-3X007T, U2 LM2596T-5, U3 ESP32-WROOM-32E, U4 LD1086DT33TR, U5 CH340C, U6 SFH617A-3X007T, U7 SFH617A-3X007T, U8 SFH617A-3X007T, U9 LM324

Commit message: added foot_prints
Parts:
- removed C22: 470u, symbol Device:C_Polarized_Small
- removed D3, D4: 1N5822, symbol Device:D_Schottky
- removed D8: MBR340, Diode_THT:D_DO-201AD_P15.24mm_Horizontal, symbol Diode:MBR340
- removed J1: USB_C_Receptacle_USB2.0_16P, Connector_USB:USB_C_Receptacle_G-Switch_GT-USB-7010ASV, symbol Connector:USB_C_Receptacle_USB2.0_16P
- removed J3: Conn_01x02_Pin, Connector_AMASS:AMASS_XT60-F_1x02_P7.20mm_Vertical, symbol Connector:Conn_01x02_Pin
- removed J4: Conn_01x05_Pin, symbol Connector:Conn_01x05_Pin
- removed SW1, SW2: SW_MEC_5G, symbol Switch:SW_MEC_5G
- added D10, D11, D13: SS34, Diode_SMD:D_SMB_Handsoldering, symbol Diode:SS34
- added D12: SS34, Diode_SMD:D_SMA_Handsoldering, symbol Diode:SS34
- added H1, H2, H3, H4: MountingHole, MountingHole:MountingHole_2.2mm_M2_ISO7380, symbol Mechanical:MountingHole
- added J1: Conn_01x06_Pin, Connector_PinHeader_2.54mm:PinHeader_1x06_P2.54mm_Vertical, symbol Connector:Conn_01x06_Pin
- added J7: USB_C_Receptacle_USB2.0_16P, Connector_USB:USB_C_Receptacle_GCT_USB4105-xx-A_16P_TopMnt_Horizontal, symbol Connector:USB_C_Receptacle_USB2.0_16P
- added SW3, SW4: SW_Push, Button_Switch_THT:SW_PUSH_6mm_H9.5mm, symbol Switch:SW_Push
- added unit 4 of U9
- C1, C11, C12, C13, C15, C17, C19, C20, C23, C25, C5, C6, C7, C8, C9: footprint (none) -> Capacitor_SMD:C_0805_2012Metric_Pad1.18x1.45mm_HandSolder
- C10, C21, C24, C3, C4: footprint (none) -> Capacitor_SMD:CP_Elec_5x4.5
- C2: footprint Connector_USB:USB_C_Receptacle_G-Switch_GT-USB-7010ASV -> Capacitor_SMD:CP_Elec_5x4.5
- D6: footprint (none) -> LED_SMD:LED_0805_2012Metric_Pad1.15x1.40mm_HandSolder
- D7, D9: footprint Diode_SMD:D_SOD-323F -> Diode_SMD:D_SOD-323_HandSoldering
- L1: footprint (none) -> Inductor_SMD:L_7.3x7.3_H4.5
- Q1: footprint (none) -> Package_TO_SOT_SMD:SOT-23-3
- R10, R11, R12, R13, R14, R15, R16, R17, R21, R22, R23, R24, R25, R26, R27, R29, R3, R30, R31, R32, R33, R34, R35, R36, R37, R39, R4, R40, R41, R42, R43, R44, R45, R46, R47, R48, R49, R5, R50, R51, R6, R7, R9: footprint (none) -> Resistor_SMD:R_0805_2012Metric_Pad1.20x1.40mm_HandSolder
- R18, R19, R20: footprint (none) -> Resistor_THT:R_Axial_DIN0614_L14.3mm_D5.7mm_P5.08mm_Vertical
- R_shunt2: footprint (none) -> Resistor_SMD:R_2512_6332Metric_Pad1.40x3.35mm_HandSolder
- TH1, TH2: footprint (none) -> Connector_PinHeader_2.54mm:PinHeader_1x02_P2.54mm_Vertical
- U11: footprint INA213AIDCKT:SOT65P210X110-6N -> Package_TO_SOT_SMD:SOT-363_SC-70-6_Handsoldering
- U4: footprint Package_TO_SOT_SMD:TO-252-2 -> Package_TO_SOT_SMD:TO-263-3_TabPin2
- U9: footprint (none) -> Package_SO:SOIC-14_3.9x8.7mm_P1.27mm
Connections:
- net +3.3V: now also J1.1 (Pin_1)
- net +5V: no longer U1.5 (VBUS)
- net C_D+: now also J7.A6 (D+), J7.B6 (D+)
- net C_D-: now also J7.A7 (D-), J7.B7 (D-)
- net EN: now also SW3.1
- net GND: now also D11.2 (A), J1.6 (Pin_6), J7.A1 (GND), J7.A12 (GND), J7.B1 (GND), J7.B12 (GND), J7.SH (SHIELD), SW3.2, SW4.2, U9.12 (+)
- net IO33: now also C25.1, D9.1 (K), R37.2, TH2.1
- net IO34: no longer C25.1, D9.1 (K), R37.2, TH2.1
- net LED1: now also U3.37 (IO23); no longer U3.28 (IO17)
- net LED2: now also U3.36 (IO22); no longer U3.27 (IO16)
- net MISO: now also J1.3 (Pin_3)
- net MOSI: now also U3.30 (IO18), J1.4 (Pin_4); no longer U3.12 (IO27)
- net SCK: now also U3.29 (IO5), J1.5 (Pin_5); no longer U3.30 (IO18)
- net V_out: now also D12.1 (K)
- net IO4: now reaches U3.26 (IO4)
- net IO4: now also R11.1
- net at R4.2: now also SW4.1
- net at C3.1, Q1.3 (S), U2.1 (VIN): now also D10.1 (K)
- net at Q1.2 (G), R3.1: now also D10.2 (A)
- net at R7.1: now also J7.B5 (CC2)
- net at R6.1: now also J7.A5 (CC1)
- net at L1.1, U2.2 (OUT): now also D11.1 (K)
- net at R27.1: now also D12.2 (A)
- net IO21 renamed CS
- net CS: now also J1.2 (Pin_2); no longer R14.1
- net IO22 renamed IO16
- net IO16: now also U3.27 (IO16); no longer U3.36 (IO22)
- removed net IO23: R11.1, U3.37 (IO23)
- new net: D13.1 (K), J7.A4 (VBUS), J7.A9 (VBUS), J7.B4 (VBUS), J7.B9 (VBUS)
- new net: U9.13 (-), U9.14
- new net 5V_USB: D13.2 (A), U1.5 (VBUS)
- new net IO17: R14.1, U3.28 (IO17)
- no-connect marks 15 -> 14

Commit message: pierwszy krok
Connections:
- net 5V_USB is gone; now on net +5V: D13.2 (A), U1.5 (VBUS)
- net IO17: now also R11.1; no longer R14.1
- net IO34: now also C13.1, R25.1, R26.2; no longer C20.1, D7.1 (K), R42.2
- net IO35: now also C20.1, D7.1 (K), R42.2; no longer C11.1, R21.1, R22.2
- net IO36: now also C11.1, R21.1, R22.2; no longer C12.1, R23.1, R24.2
- net IO39: now also C12.1, R23.1, R24.2; no longer C13.1, R25.1, R26.2
- net IO4: now also R14.1; no longer R11.1
- net V3+: now also R19.2; no longer R19.1
- net at Q5.2 (D): now also R19.1; no longer R19.2
Other:
- moved on the sheet: R19
Changed lines of the file:
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@@
 		)
 	)
-	(text_box "Main Power Distribution\n"
-		(exclude_from_sim no)
-		(at 13.97 15.24 0)
-		(size 117.475 78.74)
-		(margins 0.9525 0.9525 0.9525 0.9525)
-		(stroke
-			(width 0)
-			(type solid)
-		)
-		(fill
-			(type none)
-		)
-		(effects
-			(font
-				(size 1.27 1.27)
-				(thickness 0.254)
-				(bold yes)
-			)
-			(justify left top)
-		)
-	)
 	(text_box ""
 		(exclude_from_sim no)
@@
 	(wire
 		(pts
+			(xy 63.5 111.76) (xy 63.5 107.95)
+		)
+		(stroke
+			(width 0)
+			(type default)
+		)
+	)
+	(wire
+		(pts
 			(xy 90.17 250.19) (xy 92.71 250.19)
 		)
@@
 	(wire
 		(pts
-			(xy 57.15 111.76) (xy 58.42 111.76)
+			(xy 57.15 111.76) (xy 63.5 111.76)
 		)
 		(stroke
@@
 	(wire
 		(pts
-			(xy 68.58 132.08) (xy 68.58 135.89)
-		)
-		(stroke
-			(width 0)
-			(type default)
-		)
-	)
-	(wire
-		(pts
 			(xy 40.64 72.39) (xy 30.48 72.39)
 		)
@@
 	)
 	(label "IO34"
-		(at 341.63 227.33 0)
+		(at 220.98 260.35 0)
 		(effects
 			(font
@@
 	)
 	(label "IO39"
-		(at 220.98 260.35 0)
+		(at 222.25 224.79 0)
 		(effects
 			(font
@@
 	)
 	(label "IO4"
-		(at 125.73 265.43 0)
+		(at 127 182.88 0)
 		(effects
 			(font
@@
 	)
 	(label "IO36"
-		(at 222.25 224.79 0)
+		(at 219.71 186.69 0)
 		(effects
 			(font
@@
 	)
 	(label "IO35"
-		(at 219.71 186.69 0)
+		(at 341.63 227.33 0)
 		(effects
 			(font
@@
 		)
 	)
-	(label "5V_USB"
-		(at 58.42 111.76 0)
-		(effects
-			(font
-				(size 1.27 1.27)
-			)
-			(justify left bottom)
-		)
-	)
 	(label "V3+"
 		(at 204.47 172.72 0)
@@
 	)
 	(label "IO17"
-		(at 127 182.88 0)
+		(at 125.73 265.43 0)
 		(effects
 			(font
@@
 		)
 	)
-	(label "5V_USB"
-		(at 68.58 132.08 0)
-		(effects
-			(font
-				(size 1.27 1.27)
-			)
-			(justify left bottom)
-		)
-	)
 	(label "IO32"
 		(at 92.71 250.19 0)
@@
 	)
 	(symbol
+		(lib_id "power:+5V")
+		(at 63.5 107.95 0)
+		(unit 1)
+		(body_style 1)
+		(exclude_from_sim no)
+		(in_bom yes)
+		(on_board yes)
+		(in_pos_files yes)
+		(dnp no)
+		(fields_autoplaced yes)
+		(property "Reference" "#PWR012"
+			(at 63.5 111.76 0)
+			(hide yes)
+			(show_name no)
+			(do_not_autoplace no)
+			(effects
+				(font
+					(size 1.27 1.27)
+				)
+			)
+		)
+		(property "Value" "+5V"
+			(at 63.5 102.87 0)
+			(show_name no)
+			(do_not_autoplace no)
+			(effects
+				(font
+					(size 1.27 1.27)
+				)
+			)
+		)
+		(property "Footprint" ""
+			(at 63.5 107.95 0)
+			(hide yes)
+			(show_name no)
+			(do_not_autoplace no)
+			(effects
+				(font
+					(size 1.27 1.27)
+				)
+			)
+		)
+		(property "Datasheet" ""
+			(at 63.5 107.95 0)
+			(hide yes)
+			(show_name no)
+			(do_not_autoplace no)
+			(effects
+				(font
+					(size 1.27 1.27)
+				)
+			)
+		)
+		(property "Description" "Power symbol creates a global label with name \"+5V\""
+			(at 63.5 107.95 0)
+			(hide yes)
+			(show_name no)
+			(do_not_autoplace no)
+			(effects
+				(font
+					(size 1.27 1.27)
+				)
+			)
+		)
+		(pin "1"
+		)
+		(instances
+			(project "BMS"
+				(path "/416cad80-5d16-4386-bcbd-118262b7dc4e"
+					(reference "#PWR012")
+					(unit 1)
+				)
+			)
+		)
+	)
+	(symbol
 		(lib_id "Device:R")
 		(at 134.62 144.78 90)
@@
 	)
 	(symbol
+		(lib_id "power:+5V")
+		(at 68.58 135.89 0)
+		(unit 1)
+		(body_style 1)
+		(exclude_from_sim no)
+		(in_bom yes)
+		(on_board yes)
+		(in_pos_files yes)
+		(dnp no)
+		(property "Reference" "#PWR046"
+			(at 68.58 139.7 0)
+			(hide yes)
+			(show_name no)
+			(do_not_autoplace no)
+			(effects
+				(font
+					(size 1.27 1.27)
+				)
+			)
+		)
+		(property "Value" "+5V"
+			(at 68.58 132.334 0)
+			(show_name no)
+			(do_not_autoplace no)
+			(effects
+				(font
+					(size 1.27 1.27)
+				)
+			)
+		)
+		(property "Footprint" ""
+			(at 68.58 135.89 0)
+			(hide yes)
+			(show_name no)
+			(do_not_autoplace no)
+			(effects
+				(font
+					(size 1.27 1.27)
+				)
+			)
+		)
+		(property "Datasheet" ""
+			(at 68.58 135.89 0)
+			(hide yes)
+			(show_name no)
+			(do_not_autoplace no)
+			(effects
+				(font
+					(size 1.27 1.27)
+				)
+			)
+		)
+		(property "Description" "Power symbol creates a global label with name \"+5V\""
+			(at 68.58 135.89 0)
+			(hide yes)
+			(show_name no)
+			(do_not_autoplace no)
+			(effects
+				(font
+					(size 1.27 1.27)
+				)
+			)
+		)
+		(pin "1"
+		)
+		(instances
+			(project "BMS"
+				(path "/416cad80-5d16-4386-bcbd-118262b7dc4e"
+					(reference "#PWR046")
+					(unit 1)
+				)
+			)
+		)
+	)
+	(symbol
 		(lib_id "power:GND")
 		(at 68.58 149.86 0)
@@
 	(symbol
 		(lib_id "Device:R")
-		(at 180.34 179.07 0)
+		(at 180.34 179.07 180)
 		(unit 1)
 		(body_style 1)
@@
 		(fields_autoplaced yes)
 		(property "Reference" "R19"
-			(at 177.8 180.3401 0)
+			(at 182.88 177.7999 0)
 			(show_name no)
 			(do_not_autoplace no)
@@
 		)
 		(property "Value" "16"
-			(at 177.8 177.8001 0)
+			(at 182.88 180.3399 0)
 			(show_name no)
 			(do_not_autoplace no)
@@
 		)
 		(property "Footprint" "Resistor_THT:R_Axial_DIN0614_L14.3mm_D5.7mm_P5.08mm_Vertical"
-			(at 178.562 179.07 90)
+			(at 182.118 179.07 90)
 			(hide yes)
 			(show_name no)

Commit message: update
Connections:
- net IO17: now also R14.1; no longer R11.1
- net IO4: now also R11.1; no longer R14.1
- net V3+: now also R19.1; no longer R19.2
- net at Q5.2 (D): now also R19.2; no longer R19.1
Other:
- moved on the sheet: R19
Changed lines of the file:
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@@
 	)
 	(label "IO4"
-		(at 127 182.88 0)
+		(at 125.73 265.43 0)
 		(effects
 			(font
@@
 	)
 	(label "IO17"
-		(at 125.73 265.43 0)
+		(at 127 182.88 0)
 		(effects
 			(font
@@
 	(symbol
 		(lib_id "Device:R")
-		(at 180.34 179.07 180)
+		(at 180.34 179.07 0)
 		(unit 1)
 		(body_style 1)
@@
 					(size 1.27 1.27)
 				)
-				(justify right)
+				(justify left)
 			)
 		)
@@
 					(size 1.27 1.27)
 				)
-				(justify right)
+				(justify left)
 			)
 		)
 		(property "Footprint" "Resistor_THT:R_Axial_DIN0614_L14.3mm_D5.7mm_P5.08mm_Vertical"
-			(at 182.118 179.07 90)
+			(at 178.562 179.07 90)
 			(hide yes)
 			(show_name no)

Commit message: linki do TME
Parts:
- removed D7, D9: MM3Zxx, Diode_SMD:D_SOD-323_HandSoldering, symbol Diode:MM3Zxx
- added D7, D8: D_Zener, Diode_SMD:D_SOD-323_HandSoldering, symbol Device:D_Zener
- D12: footprint Diode_SMD:D_SMA_Handsoldering -> Diode_SMD:D_SMB_Handsoldering
Connections:
- net GND: now also D7.2 (A), D8.2 (A)
- net IO33: now also D8.1 (K)
- net IO35: now also D7.1 (K)
Changed lines of the file:
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@@
 	)
 	(symbol
-		(lib_id "Diode:MM3Zxx")
-		(at 321.31 236.22 270)
-		(unit 1)
-		(body_style 1)
-		(exclude_from_sim no)
-		(in_bom yes)
-		(on_board yes)
-		(in_pos_files yes)
-		(dnp no)
-		(fields_autoplaced yes)
-		(property "Reference" "D7"
-			(at 323.85 234.9499 90)
-			(show_name no)
-			(do_not_autoplace no)
-			(effects
-				(font
-					(size 1.27 1.27)
-				)
-				(justify left)
-			)
-		)
-		(property "Value" "MM3Zxx"
-			(at 323.85 237.4899 90)
-			(show_name no)
-			(do_not_autoplace no)
-			(effects
-				(font
-					(size 1.27 1.27)
-				)
-				(justify left)
-			)
-		)
-		(property "Footprint" "Diode_SMD:D_SOD-323_HandSoldering"
-			(at 316.865 236.22 0)
-			(hide yes)
-			(show_name no)
-			(do_not_autoplace no)
-			(effects
-				(font
-					(size 1.27 1.27)
-				)
-			)
-		)
-		(property "Datasheet" "https://diotec.com/tl_files/diotec/files/pdf/datasheets/mm3z2v4.pdf"
-			(at 321.31 236.22 0)
-			(hide yes)
-			(show_name no)
-			(do_not_autoplace no)
-			(effects
-				(font
-					(size 1.27 1.27)
-				)
-			)
-		)
-		(property "Description" "300mW Zener Diode, SOD-323F"
-			(at 321.31 236.22 0)
-			(hide yes)
-			(show_name no)
-			(do_not_autoplace no)
-			(effects
-				(font
-					(size 1.27 1.27)
-				)
-			)
-		)
-		(pin "1"
-		)
-		(pin "2"
-		)
-		(instances
-			(project "BMS"
-				(path "/416cad80-5d16-4386-bcbd-118262b7dc4e"
-					(reference "D7")
-					(unit 1)
-				)
-			)
-		)
-	)
-	(symbol
 		(lib_id "Interface_USB:CH340C")
 		(at 100.33 130.81 0)
@@
 			)
 		)
-		(property "Footprint" "Diode_SMD:D_SMA_Handsoldering"
+		(property "Footprint" "Diode_SMD:D_SMB_Handsoldering"
 			(at 387.985 26.67 0)
 			(hide yes)
@@
 	)
 	(symbol
+		(lib_id "Device:D_Zener")
+		(at 321.31 236.22 270)
+		(unit 1)
+		(body_style 1)
+		(exclude_from_sim no)
+		(in_bom yes)
+		(on_board yes)
+		(in_pos_files yes)
+		(dnp no)
+		(fields_autoplaced yes)
+		(property "Reference" "D7"
+			(at 323.85 234.9499 90)
+			(show_name no)
+			(do_not_autoplace no)
+			(effects
+				(font
+					(size 1.27 1.27)
+				)
+				(justify left)
+			)
+		)
+		(property "Value" "D_Zener"
+			(at 323.85 237.4899 90)
+			(show_name no)
+			(do_not_autoplace no)
+			(effects
+				(font
+					(size 1.27 1.27)
+				)
+				(justify left)
+			)
+		)
+		(property "Footprint" "Diode_SMD:D_SOD-323_HandSoldering"
+			(at 321.31 236.22 0)
+			(hide yes)
+			(show_name no)
+			(do_not_autoplace no)
+			(effects
+				(font
+					(size 1.27 1.27)
+				)
+			)
+		)
+		(property "Datasheet" ""
+			(at 321.31 236.22 0)
+			(hide yes)
+			(show_name no)
+			(do_not_autoplace no)
+			(effects
+				(font
+					(size 1.27 1.27)
+				)
+			)
+		)
+		(property "Description" "Zener diode"
+			(at 321.31 236.22 0)
+			(hide yes)
+			(show_name no)
+			(do_not_autoplace no)
+			(effects
+				(font
+					(size 1.27 1.27)
+				)
+			)
+		)
+		(pin "1"
+		)
+		(pin "2"
+		)
+		(instances
+			(project "BMS"
+				(path "/416cad80-5d16-4386-bcbd-118262b7dc4e"
+					(reference "D7")
+					(unit 1)
+				)
+			)
+		)
+	)
+	(symbol
 		(lib_id "Device:C")
 		(at 63.5 175.26 0)
@@
 	)
 	(symbol
+		(lib_id "Device:D_Zener")
+		(at 201.93 134.62 270)
+		(unit 1)
+		(body_style 1)
+		(exclude_from_sim no)
+		(in_bom yes)
+		(on_board yes)
+		(in_pos_files yes)
+		(dnp no)
+		(fields_autoplaced yes)
+		(property "Reference" "D8"
+			(at 204.47 133.3499 90)
+			(show_name no)
+			(do_not_autoplace no)
+			(effects
+				(font
+					(size 1.27 1.27)
+				)
+				(justify left)
+			)
+		)
+		(property "Value" "D_Zener"
+			(at 204.47 135.8899 90)
+			(show_name no)
+			(do_not_autoplace no)
+			(effects
+				(font
+					(size 1.27 1.27)
+				)
+				(justify left)
+			)
+		)
+		(property "Footprint" "Diode_SMD:D_SOD-323_HandSoldering"
+			(at 201.93 134.62 0)
+			(hide yes)
+			(show_name no)
+			(do_not_autoplace no)
+			(effects
+				(font
+					(size 1.27 1.27)
+				)
+			)
+		)
+		(property "Datasheet" ""
+			(at 201.93 134.62 0)
+			(hide yes)
+			(show_name no)
+			(do_not_autoplace no)
+			(effects
+				(font
+					(size 1.27 1.27)
+				)
+			)
+		)
+		(property "Description" "Zener diode"
+			(at 201.93 134.62 0)
+			(hide yes)
+			(show_name no)
+			(do_not_autoplace no)
+			(effects
+				(font
+					(size 1.27 1.27)
+				)
+			)
+		)
+		(pin "1"
+		)
+		(pin "2"
+		)
+		(instances
+			(project "BMS"
+				(path "/416cad80-5d16-4386-bcbd-118262b7dc4e"
+					(reference "D8")
+					(unit 1)
+				)
+			)
+		)
+	)
+	(symbol
 		(lib_id "Device:C_Polarized_Small")
 		(at 401.32 199.39 0)
@@
 					(unit 1)
 				)
-			)
-		)
-	)
-	(symbol
-		(lib_id "Diode:MM3Zxx")
-		(at 201.93 134.62 270)
-		(unit 1)
-		(body_style 1)
-		(exclude_from_sim no)
-		(in_bom yes)
-		(on_board yes)
-		(in_pos_files yes)
-		(dnp no)
-		(fields_autoplaced yes)
-		(property "Reference" "D9"
-			(at 204.47 133.3499 90)
-			(show_name no)
-			(do_not_autoplace no)
-			(effects
-				(font
-					(size 1.27 1.27)
-				)
-				(justify left)
-			)
-		)
-		(property "Value" "MM3Zxx"
-			(at 204.47 135.8899 90)
-			(show_name no)
-			(do_not_autoplace no)
-			(effects
-				(font
-					(size 1.27 1.27)
-				)
-				(justify left)
-			)
-		)
-		(property "Footprint" "Diode_SMD:D_SOD-323_HandSoldering"
-			(at 197.485 134.62 0)
-			(hide yes)
-			(show_name no)
-			(do_not_autoplace no)
-			(effects
-				(font
-					(size 1.27 1.27)
-				)
-			)
-		)
-		(property "Datasheet" "https://diotec.com/tl_files/diotec/files/pdf/datasheets/mm3z2v4.pdf"
-			(at 201.93 134.62 0)
-			(hide yes)
-			(show_name no)
-			(do_not_autoplace no)
-			(effects
-				(font
-					(size 1.27 1.27)
-				)
-			)
-		)
-		(property "Description" "300mW Zener Diode, SOD-323F"
-			(at 201.93 134.62 0)
-			(hide yes)
-			(show_name no)
-			(do_not_autoplace no)
-			(effects
-				(font
-					(size 1.27 1.27)
-				)
-			)
-		)
-		(pin "1"
-		)
-		(pin "2"
-		)
-		(instances
-			(project "BMS"
-				(path "/416cad80-5d16-4386-bcbd-118262b7dc4e"
-					(reference "D9")
-					(unit 1)
-				)

Commit message: update
Connections:
- net IO25: now also R43.2; no longer R44.2
- net IO26: now also R44.2; no longer R43.2
- net IO32: now also C25.1, D8.1 (K), R37.2, TH2.1; no longer C19.1, R39.2, R40.1
- net IO33: now also C19.1, R39.2, R40.1; no longer C25.1, D8.1 (K), R37.2, TH2.1
Changed lines of the file:
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@@
 	)
 	(label "IO26"
-		(at 308.61 77.47 180)
+		(at 308.61 33.02 180)
 		(effects
 			(font
@@
 	)
 	(label "IO33"
-		(at 222.25 125.73 180)
+		(at 293.37 64.77 180)
 		(effects
 			(font
@@
 	)
 	(label "IO25"
-		(at 308.61 33.02 180)
+		(at 308.61 77.47 180)
 		(effects
 			(font
@@
 	)
 	(label "IO32"
-		(at 293.37 64.77 0)
-		(effects
-			(font
+		(at 222.25 125.73 0)
+		(effects
+			(font
