File: BMS.kicad_sch (KiCad schematic)
At the start: 119 parts, among them J1 Conn_01x06_Pin, J2 Conn_01x02_Pin, J5 Conn_01x02_Pin, J6 Conn_01x04_Pin, J7 USB_C_Receptacle_USB2.0_16P, Q1 MMFTP3401-AQ, Q2 2N7002, Q3 SS8050, Q4 IRLZ44N, Q5 IRLZ44N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

Commit message: poprawa
Parts:
- L1: value 47u -> 33u
Connections:
- net GND: now also D12.2 (A)
- net V_out: now also R27.1
Other:
- moved on the sheet: R27
Changed lines of the file:
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@@
 	)
 	(junction
+		(at 383.54 20.32)
+		(diameter 0)
+		(color 0 0 0 0)
+	)
+	(junction
 		(at 372.11 90.17)
 		(diameter 0)
@@
 	)
 	(junction
+		(at 392.43 43.18)
+		(diameter 0)
+		(color 0 0 0 0)
+	)
+	(junction
 		(at 88.9 68.58)
 		(diameter 0)
@@
 	(wire
 		(pts
+			(xy 383.54 20.32) (xy 392.43 20.32)
+		)
+		(stroke
+			(width 0)
+			(type default)
+		)
+	)
+	(wire
+		(pts
 			(xy 370.84 170.18) (xy 370.84 171.45)
 		)
@@
 	(wire
 		(pts
-			(xy 392.43 30.48) (xy 392.43 33.02)
-		)
-		(stroke
-			(width 0)
-			(type default)
-		)
-	)
-	(wire
-		(pts
 			(xy 73.66 143.51) (xy 74.93 143.51)
 		)
@@
 	(wire
 		(pts
-			(xy 372.11 20.32) (xy 392.43 20.32)
+			(xy 372.11 20.32) (xy 383.54 20.32)
 		)
 		(stroke
@@
 	(wire
 		(pts
+			(xy 392.43 43.18) (xy 392.43 44.45)
+		)
+		(stroke
+			(width 0)
+			(type default)
+		)
+	)
+	(wire
+		(pts
 			(xy 218.44 186.69) (xy 219.71 186.69)
 		)
@@
 	(wire
 		(pts
+			(xy 392.43 30.48) (xy 392.43 43.18)
+		)
+		(stroke
+			(width 0)
+			(type default)
+		)
+	)
+	(wire
+		(pts
 			(xy 115.57 69.85) (xy 115.57 68.58)
 		)
@@
 	(wire
 		(pts
-			(xy 392.43 40.64) (xy 392.43 44.45)
+			(xy 383.54 31.75) (xy 383.54 43.18)
 		)
 		(stroke
@@
 	(wire
 		(pts
+			(xy 383.54 20.32) (xy 383.54 24.13)
+		)
+		(stroke
+			(width 0)
+			(type default)
+		)
+	)
+	(wire
+		(pts
 			(xy 349.25 27.94) (xy 349.25 33.02)
 		)
@@
 	(wire
 		(pts
+			(xy 383.54 43.18) (xy 392.43 43.18)
+		)
+		(stroke
+			(width 0)
+			(type default)
+		)
+	)
+	(wire
+		(pts
 			(xy 398.78 20.32) (xy 392.43 20.32)
 		)
@@
 			)
 		)
-		(property "Value" "47u"
+		(property "Value" "33u"
 			(at 95.25 66.04 90)
 			(show_name no)
@@
 	(symbol
 		(lib_id "Device:R")
-		(at 392.43 36.83 0)
+		(at 383.54 27.94 0)
 		(unit 1)
 		(body_style 1)
@@
 		(fields_autoplaced yes)
 		(property "Reference" "R27"
-			(at 394.97 35.5599 0)
+			(at 386.08 26.6699 0)
 			(show_name no)
 			(do_not_autoplace no)
@@
 		)
 		(property "Value" "1k"
-			(at 394.97 38.0999 0)
+			(at 386.08 29.2099 0)
 			(show_name no)
 			(do_not_autoplace no)
@@
 		)
 		(property "Footprint" "Resistor_SMD:R_0805_2012Metric_Pad1.20x1.40mm_HandSolder"
-			(at 390.652 36.83 90)
+			(at 381.762 27.94 90)
 			(hide yes)
 			(show_name no)
@@
 		)
 		(property "Datasheet" ""
-			(at 392.43 36.83 0)
+			(at 383.54 27.94 0)
 			(hide yes)
 			(show_name no)
@@
 		)
 		(property "Description" "Resistor"
-			(at 392.43 36.83 0)
+			(at 383.54 27.94 0)
 			(hide yes)
 			(show_name no)

Commit message: Dioda
Connections:
- net +5V: now also D13.1 (K); no longer D13.2 (A)
- net at J7.A4 (VBUS), J7.A9 (VBUS), J7.B4 (VBUS)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: now also D13.2 (A); no longer D13.1 (K)
Other:
- moved on the sheet: D13
Changed lines of the file:
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@@
 	(symbol
 		(lib_id "Diode:SS34")
-		(at 53.34 111.76 0)
+		(at 53.34 111.76 180)
 		(unit 1)
 		(body_style 1)
@@
 		(fields_autoplaced yes)
 		(property "Reference" "D13"
-			(at 53.0225 105.41 0)
+			(at 53.6575 105.41 0)
 			(show_name no)
 			(do_not_autoplace no)
@@
 		)
 		(property "Value" "SS34"
-			(at 53.0225 107.95 0)
+			(at 53.6575 107.95 0)
 			(show_name no)
 			(do_not_autoplace no)
@@
 		)
 		(property "Footprint" "Diode_SMD:D_SMB_Handsoldering"
-			(at 53.34 116.205 0)
+			(at 53.34 107.315 0)
 			(hide yes)
 			(show_name no)

Commit message: KOndensator
Parts:
- added C14: 100n, Capacitor_SMD:C_0805_2012Metric_Pad1.18x1.45mm_HandSolder, symbol Device:C
Connections:
- net +5V: now also C14.1
- net GND: now also C14.2
Changed lines of the file:
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@@
 	(text_box "ESP32 Programming Section\n"
 		(exclude_from_sim no)
-		(at 15.24 96.52 0)
+		(at 14.986 97.536 0)
 		(size 147.32 60.96)
 		(margins 0.9525 0.9525 0.9525 0.9525)
@@
 	)
 	(junction
+		(at 68.58 149.86)
+		(diameter 0)
+		(color 0 0 0 0)
+	)
+	(junction
 		(at 261.62 35.56)
 		(diameter 0)
@@
 	)
 	(junction
+		(at 68.58 135.89)
+		(diameter 0)
+		(color 0 0 0 0)
+	)
+	(junction
 		(at 379.73 224.79)
 		(diameter 0)
@@
 	(wire
 		(pts
+			(xy 68.58 135.89) (xy 83.82 135.89)
+		)
+		(stroke
+			(width 0)
+			(type default)
+		)
+	)
+	(wire
+		(pts
 			(xy 92.71 245.11) (xy 90.17 245.11)
 		)
@@
 	(wire
 		(pts
+			(xy 68.58 149.86) (xy 83.82 149.86)
+		)
+		(stroke
+			(width 0)
+			(type default)
+		)
+	)
+	(wire
+		(pts
 			(xy 120.65 127) (xy 130.81 127)
 		)
@@
 	(wire
 		(pts
+			(xy 68.58 134.62) (xy 68.58 135.89)
+		)
+		(stroke
+			(width 0)
+			(type default)
+		)
+	)
+	(wire
+		(pts
 			(xy 284.48 160.02) (xy 288.29 160.02)
 		)
@@
 	(wire
 		(pts
+			(xy 68.58 149.86) (xy 68.58 148.59)
+		)
+		(stroke
+			(width 0)
+			(type default)
+		)
+	)
+	(wire
+		(pts
 			(xy 209.55 247.65) (xy 208.28 247.65)
 		)
@@
 	(wire
 		(pts
-			(xy 68.58 149.86) (xy 68.58 148.59)
+			(xy 68.58 151.13) (xy 68.58 149.86)
 		)
 		(stroke
@@
 	(wire
 		(pts
+			(xy 83.82 138.43) (xy 83.82 135.89)
+		)
+		(stroke
+			(width 0)
+			(type default)
+		)
+	)
+	(wire
+		(pts
 			(xy 236.22 210.82) (xy 245.11 210.82)
 		)
@@
 	(wire
 		(pts
+			(xy 83.82 149.86) (xy 83.82 146.05)
+		)
+		(stroke
+			(width 0)
+			(type default)
+		)
+	)
+	(wire
+		(pts
 			(xy 17.78 60.96) (xy 17.78 63.5)
 		)
@@
 		(in_pos_files yes)
 		(dnp no)
-		(fields_autoplaced yes)
 		(property "Reference" "U1"
 			(at 70.2311 133.35 0)
@@
 		)
 		(property "Value" "USBLC6-2SC6"
-			(at 70.2311 135.89 0)
+			(at 68.58 137.414 0)
 			(show_name no)
 			(do_not_autoplace no)
@@
 	(symbol
 		(lib_id "power:+5V")
-		(at 68.58 135.89 0)
+		(at 68.58 134.62 0)
 		(unit 1)
 		(body_style 1)
@@
 		(dnp no)
 		(property "Reference" "#PWR046"
-			(at 68.58 139.7 0)
+			(at 68.58 138.43 0)
 			(hide yes)
 			(show_name no)
@@
 		)
 		(property "Value" "+5V"
-			(at 68.58 132.334 0)
+			(at 68.58 131.064 0)
 			(show_name no)
 			(do_not_autoplace no)
@@
 		)
 		(property "Footprint" ""
-			(at 68.58 135.89 0)
+			(at 68.58 134.62 0)
 			(hide yes)
 			(show_name no)
@@
 		)
 		(property "Datasheet" ""
-			(at 68.58 135.89 0)
+			(at 68.58 134.62 0)
 			(hide yes)
 			(show_name no)
@@
 		)
 		(property "Description" "Power symbol creates a global label with name \"+5V\""
-			(at 68.58 135.89 0)
+			(at 68.58 134.62 0)
 			(hide yes)
 			(show_name no)
@@
 	(symbol
 		(lib_id "power:GND")
-		(at 68.58 149.86 0)
+		(at 68.58 151.13 0)
 		(unit 1)
 		(body_style 1)
@@
 		(fields_autoplaced yes)
 		(property "Reference" "#PWR014"
-			(at 68.58 156.21 0)
+			(at 68.58 157.48 0)
 			(hide yes)
 			(show_name no)
@@
 		)
 		(property "Value" "GND"
-			(at 68.58 154.94 0)
+			(at 68.58 156.21 0)
 			(show_name no)
 			(do_not_autoplace no)
@@
 		)
 		(property "Footprint" ""
-			(at 68.58 149.86 0)
+			(at 68.58 151.13 0)
 			(hide yes)
 			(show_name no)
@@
 		)
 		(property "Datasheet" ""
-			(at 68.58 149.86 0)
+			(at 68.58 151.13 0)
 			(hide yes)
 			(show_name no)
@@
 		)
 		(property "Description" "Power symbol creates a global label with name \"GND\" , ground"
-			(at 68.58 149.86 0)
+			(at 68.58 151.13 0)
 			(hide yes)
 			(show_name no)
@@
 					(unit 1)
 				)
+			)
+		)
+	)
+	(symbol
+		(lib_id "Device:C")
+		(at 83.82 142.24 0)
+		(unit 1)
+		(body_style 1)
+		(exclude_from_sim no)
+		(in_bom yes)
+		(on_board yes)
+		(in_pos_files yes)
+		(dnp no)
+		(fields_autoplaced yes)
+		(property "Reference" "C14"
+			(at 87.63 140.9699 0)
+			(show_name no)
+			(do_not_autoplace no)
+			(effects
+				(font
+					(size 1.27 1.27)
+				)
+				(justify left)
+			)
+		)
+		(property "Value" "100n"
+			(at 87.63 143.5099 0)
+			(show_name no)
+			(do_not_autoplace no)
+			(effects
+				(font
+					(size 1.27 1.27)
+				)
+				(justify left)
+			)
+		)
+		(property "Footprint" "Capacitor_SMD:C_0805_2012Metric_Pad1.18x1.45mm_HandSolder"
+			(at 84.7852 146.05 0)
+			(hide yes)
+			(show_name no)
+			(do_not_autoplace no)
+			(effects
+				(font
+					(size 1.27 1.27)
+				)
+			)
+		)
+		(property "Datasheet" ""
+			(at 83.82 142.24 0)
+			(hide yes)
+			(show_name no)
+			(do_not_autoplace no)
+			(effects
+				(font
+					(size 1.27 1.27)
+				)
+			)
+		)
+		(property "Description" "Unpolarized capacitor"
+			(at 83.82 142.24 0)
+			(hide yes)
+			(show_name no)
+			(do_not_autoplace no)
+			(effects
+				(font
+					(size 1.27 1.27)
+				)
+			)
+		)
+		(pin "2"
+		)
+		(pin "1"
+		)
+		(instances
+			(project "BMS"
+				(path "/416cad80-5d16-4386-bcbd-118262b7dc4e"
+					(reference "C14")
+					(unit 1)
+				)

Commit message: rezystor V_out
Parts:
- removed R27: 1k, Resistor_SMD:R_0805_2012Metric_Pad1.20x1.40mm_HandSolder, symbol Device:R
Changed lines of the file:
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@@
 	)
 	(junction
-		(at 383.54 20.32)
-		(diameter 0)
-		(color 0 0 0 0)
-	)
-	(junction
 		(at 372.11 90.17)
 		(diameter 0)
@@
 	)
 	(junction
-		(at 392.43 43.18)
-		(diameter 0)
-		(color 0 0 0 0)
-	)
-	(junction
 		(at 88.9 68.58)
 		(diameter 0)
@@
 	(wire
 		(pts
-			(xy 383.54 20.32) (xy 392.43 20.32)
+			(xy 372.11 20.32) (xy 392.43 20.32)
 		)
 		(stroke
@@
 	(wire
 		(pts
-			(xy 372.11 20.32) (xy 383.54 20.32)
-		)
-		(stroke
-			(width 0)
-			(type default)
-		)
-	)
-	(wire
-		(pts
 			(xy 361.95 33.02) (xy 364.49 33.02)
 		)
@@
 	(wire
 		(pts
-			(xy 392.43 43.18) (xy 392.43 44.45)
+			(xy 392.43 30.48) (xy 392.43 44.45)
 		)
 		(stroke
@@
 	(wire
 		(pts
-			(xy 392.43 30.48) (xy 392.43 43.18)
-		)
-		(stroke
-			(width 0)
-			(type default)
-		)
-	)
-	(wire
-		(pts
 			(xy 115.57 69.85) (xy 115.57 68.58)
 		)
@@
 	(wire
 		(pts
-			(xy 383.54 31.75) (xy 383.54 43.18)
-		)
-		(stroke
-			(width 0)
-			(type default)
-		)
-	)
-	(wire
-		(pts
 			(xy 90.17 207.01) (xy 92.71 207.01)
 		)
@@
 	(wire
 		(pts
-			(xy 383.54 20.32) (xy 383.54 24.13)
-		)
-		(stroke
-			(width 0)
-			(type default)
-		)
-	)
-	(wire
-		(pts
 			(xy 349.25 27.94) (xy 349.25 33.02)
 		)
@@
 	(wire
 		(pts
-			(xy 383.54 43.18) (xy 392.43 43.18)
-		)
-		(stroke
-			(width 0)
-			(type default)
-		)
-	)
-	(wire
-		(pts
 			(xy 398.78 20.32) (xy 392.43 20.32)
 		)
@@
 					(unit 1)
 				)
-			)
-		)
-	)
-	(symbol
-		(lib_id "Device:R")
-		(at 383.54 27.94 0)
-		(unit 1)
-		(body_style 1)
-		(exclude_from_sim no)
-		(in_bom yes)
-		(on_board yes)
-		(in_pos_files yes)
-		(dnp no)
-		(fields_autoplaced yes)
-		(property "Reference" "R27"
-			(at 386.08 26.6699 0)
-			(show_name no)
-			(do_not_autoplace no)
-			(effects
-				(font
-					(size 1.27 1.27)
-				)
-				(justify left)
-			)
-		)
-		(property "Value" "1k"
-			(at 386.08 29.2099 0)
-			(show_name no)
-			(do_not_autoplace no)
-			(effects
-				(font
-					(size 1.27 1.27)
-				)
-				(justify left)
-			)
-		)
-		(property "Footprint" "Resistor_SMD:R_0805_2012Metric_Pad1.20x1.40mm_HandSolder"
-			(at 381.762 27.94 90)
-			(hide yes)
-			(show_name no)
-			(do_not_autoplace no)
-			(effects
-				(font
-					(size 1.27 1.27)
-				)
-			)
-		)
-		(property "Datasheet" ""
-			(at 383.54 27.94 0)
-			(hide yes)
-			(show_name no)
-			(do_not_autoplace no)
-			(effects
-				(font
-					(size 1.27 1.27)
-				)
-			)
-		)
-		(property "Description" "Resistor"
-			(at 383.54 27.94 0)
-			(hide yes)
-			(show_name no)
-			(do_not_autoplace no)
-			(effects
-				(font
-					(size 1.27 1.27)
-				)
-			)
-		)
-		(pin "1"
-		)
-		(pin "2"
-		)
-		(instances
-			(project "BMS"
-				(path "/416cad80-5d16-4386-bcbd-118262b7dc4e"
-					(reference "R27")
-					(unit 1)
-				)

Commit message: poprawiłem
Parts:
- removed C1: 100n, Capacitor_SMD:C_0805_2012Metric_Pad1.18x1.45mm_HandSolder, symbol Device:C
- removed C6, C9: 10u, Capacitor_SMD:C_0805_2012Metric_Pad1.18x1.45mm_HandSolder, symbol Device:C
- added C16, C18: 100n, Capacitor_SMD:C_0805_2012Metric_Pad1.18x1.45mm_HandSolder, symbol Device:C
- added C26, C27: 10u, Capacitor_SMD:CP_Elec_5x4.5, symbol Device:C_Polarized
- added C28: 100n, Capacitor_SMD:C_0603_1608Metric, symbol Device:C
- added R27: 10k, Resistor_SMD:R_0805_2012Metric_Pad1.20x1.40mm_HandSolder, symbol Device:R
- C2: value 22u -> 100n
- L1: footprint Inductor_SMD:L_7.3x7.3_H4.5 -> Inductor_SMD:L_Panasonic_PCC-M0630M
Connections:
- net +3.3V: now also U5.4 (V3), C27.1, R27.1
- net +5V: now also C18.1, C26.1
- net +BATT: now also C16.1
- net GND: now also C16.2, C18.2, C26.2, C27.2, C28.2
- net at R4.2, SW4.1: now also C28.1, R27.2
- no-connect marks 13 -> 12
Other:
- moved on the sheet: D10, SW3, SW4
