File: BMS.kicad_pcb (KiCad board)
At the start: 4 copper layers, 86 x 86 mm, 116 parts, among them J1 Conn_01x06_Pin, J2 Conn_01x02_Pin, J5 Conn_01x02_Pin, J6 Conn_01x04_Pin, J7 USB_C_Receptacle_USB2.0_16P, Q1 MMFTP3401-AQ, Q3 SS8050, Q4 IRLZ44N, Q5 IRLZ44N, Q6 IRLZ44N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

Commit message: Dodanie resystora do PT100
Parts:
- added Q2: 2N7002, Package_TO_SOT_SMD:SOT-23_Handsoldering, B.Cu at (67.4, 54.7)
- added R28: 2000, Resistor_SMD:R_0805_2012Metric_Pad1.20x1.40mm_HandSolder, B.Cu at (72.0, 50.7)
- added R52: 100, Resistor_SMD:R_0805_2012Metric_Pad1.20x1.40mm_HandSolder, B.Cu at (68.9, 50.7)
- R8: moved to F.Cu
Connections:
- R32 pad 2: GND -> Net-(Q2-D)
- TH1 pad 2: GND -> Net-(Q2-D)
- U3 pad 16: unconnected-(U3-IO13-Pad16) -> /IO13
Routing:
- net Net-(Q2-D): track 0.00 -> 19.7 mm, vias 0 -> 1
- net /IO13: track 0.00 -> 8.95 mm, vias 0 -> 1
- net Net-(Q2-G): track 0.00 -> 2.05 mm
- net Net-(D5-A): vias 1 -> 0
- net GND: vias 192 -> 218

Commit message: update0.4
Parts:
- C25, D8, R37: moved to F.Cu
- moved C20 4.25 mm to (48.9, 46.4)
- moved D7 4.25 mm to (48.7, 49.2)
- moved R42 4.25 mm to (49.0, 51.9)
- moved D8 0.57 mm to (55.0, 50.3)
- moved C25 0.54 mm to (55.2, 47.6)
Routing:
- net /IO35: track 17.9 -> 22.4 mm
- net Net-(R41-Pad2): track 18.9 -> 14.8 mm
- net /IO32: track 23.3 -> 23.0 mm, vias 1 -> 0
- net +3.3V: track 137.0 -> 137.2 mm, vias 7 -> 8
- net GND: vias 218 -> 214

Commit message: L1_47u
Parts:
- L1: value 33u -> 47u
Changed lines of the file:
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@@
 			)
 		)
-		(property "Value" "33u"
+		(property "Value" "47u"
 			(at 0 -4.45 0)
 			(layer "B.Fab")
@@
 	)
 	(segment
+		(start 56.2675 47.63)
+		(end 56.2375 47.6)
+		(width 0.3)
+		(layer "F.Cu")
+		(net "/IO32")
+	)
+	(segment
+		(start 56.2275 47.8575)
+		(end 56.2275 40.9325)
+		(width 0.3)
+		(layer "F.Cu")
+		(net "/IO32")
+	)
+	(segment
+		(start 56.2675 51.7075)
+		(end 56.2675 50.29)
+		(width 0.3)
+		(layer "F.Cu")
+		(net "/IO32")
+	)
+	(segment
+		(start 56.2275 40.9325)
+		(end 60.2 36.96)
+		(width 0.3)
+		(layer "F.Cu")
+		(net "/IO32")
+	)
+	(segment
+		(start 56.2675 50.29)
+		(end 56.2675 47.63)
+		(width 0.3)
+		(layer "F.Cu")
+		(net "/IO32")
+	)
+	(segment
+		(start 56.73 52.17)
+		(end 56.2675 51.7075)
+		(width 0.3)
+		(layer "F.Cu")
+		(net "/IO32")
+	)
+	(segment
+		(start 56.73 53.38)
+		(end 56.73 52.17)
+		(width 0.3)
+		(layer "F.Cu")
+		(net "/IO32")
+	)
+	(segment
+		(start 56.735 56.76)
+		(end 56.735 53.385)
+		(width 0.3)
+		(layer "F.Cu")
+		(net "/IO32")
+	)
+	(segment
+		(start 60.2 36.96)
+		(end 61.25 36.96)
+		(width 0.3)
+		(layer "F.Cu")
+		(net "/IO32")
+	)
+	(segment
 		(start 89.54 81.51)
 		(end 87.6 81.51)
@@
 	)
 	(segment
-		(start 56.2675 47.63)
-		(end 56.2375 47.6)
-		(width 0.3)
-		(layer "F.Cu")
-		(net "/IO32")
-	)
-	(segment
-		(start 56.2275 47.8575)
-		(end 56.2275 40.9325)
-		(width 0.3)
-		(layer "F.Cu")
-		(net "/IO32")
-	)
-	(segment
-		(start 56.2675 51.7075)
-		(end 56.2675 50.29)
-		(width 0.3)
-		(layer "F.Cu")
-		(net "/IO32")
-	)
-	(segment
-		(start 56.2275 40.9325)
-		(end 60.2 36.96)
-		(width 0.3)
-		(layer "F.Cu")
-		(net "/IO32")
-	)
-	(segment
-		(start 56.2675 50.29)
-		(end 56.2675 47.63)
-		(width 0.3)
-		(layer "F.Cu")
-		(net "/IO32")
-	)
-	(segment
-		(start 56.73 52.17)
-		(end 56.2675 51.7075)
-		(width 0.3)
-		(layer "F.Cu")
-		(net "/IO32")
-	)
-	(segment
-		(start 56.73 53.38)
-		(end 56.73 52.17)
-		(width 0.3)
-		(layer "F.Cu")
-		(net "/IO32")
-	)
-	(segment
-		(start 56.735 56.76)
-		(end 56.735 53.385)
-		(width 0.3)
-		(layer "F.Cu")
-		(net "/IO32")
-	)
-	(segment
-		(start 60.2 36.96)
-		(end 61.25 36.96)
-		(width 0.3)
-		(layer "F.Cu")
-		(net "/IO32")
-	)
-	(segment

Commit message: poprawa
Parts:
- L1: value 47u -> 33u
- moved R27 17.4 mm to (66.7, 109.9), turned to 180 degrees
- moved D11 13.5 mm to (31.4, 101.1), turned to -90 degrees
- moved C3 9.42 mm to (50.0, 100.1)
- moved D10 8.66 mm to (45.5, 92.9)
- moved R3 7.93 mm to (37.6, 93.0), turned to 180 degrees
- moved Q1 2.05 mm to (43.9, 99.1), turned to 0 degrees
- moved C10 1.57 mm to (47.1, 84.1)
- moved L1 1.13 mm to (31.2, 90.5), turned to 90 degrees
- moved C17 0.94 mm to (48.5, 86.8), turned to 90 degrees
Connections:
- D12 pad 2: Net-(D12-A) -> GND
- R27 pad 1: Net-(D12-A) -> /V_out
Routing:
- net Net-(D10-K): track 40.2 -> 0.00 mm
- net +5V: track 184.4 -> 171.0 mm
- net Net-(D11-K): track 11.1 -> 0.20 mm
- net Net-(D12-A): track 5.71 -> 0.00 mm
- net Net-(D10-A): track 5.68 -> 0.00 mm
- net +BATT: track 23.3 -> 18.2 mm
- net /V_out: track 21.8 -> 26.3 mm
- net GND: track 15.6 -> 19.3 mm, vias 214 -> 213
- net /V2+: track 114.1 -> 115.4 mm
- net /V1+: track 100.4 -> 101.5 mm
- net /V3+: track 113.3 -> 114.4 mm
- added copper zone on B.Cu, net +5V
- added copper zone on B.Cu, net +BATT
- added copper zone on B.Cu, net Net-(D10-A)
- added copper zone on B.Cu, net Net-(D10-K)
- added copper zone on B.Cu, net Net-(D11-K)

Commit message: przetwornica
Parts:
- moved D11 1.43 mm to (31.3, 99.7)
- moved C3 1.03 mm to (49.1, 100.7)
Changed lines of the file:
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@@
 	(footprint "Diode_SMD:D_SMB_Handsoldering"
 		(layer "B.Cu")
-		(at 31.41 101.14 -90)
+		(at 31.29 99.72 -90)
 		(descr "Diode SMB (DO-214AA) Handsoldering")
 		(tags "Diode SMB (DO-214AA) Handsoldering")
@@
 		(tags "SOT TO_SOT_SMD")
 		(property "Reference" "Q1"
-			(at 2.1 1.14 0)
+			(at -0.1875 2.44 0)
 			(layer "B.SilkS")
 			(effects
@@
 	(footprint "Capacitor_SMD:CP_Elec_5x4.5"
 		(layer "B.Cu")
-		(at 49.96 100.13 -90)
+		(at 49.07 100.65 -90)
 		(descr "SMD capacitor, aluminum electrolytic, Nichicon, 5.0x4.5mm")
 		(tags "capacitor electrolytic")
@@
 	)
 	(segment
+		(start 67.65 109.86)
+		(end 72.1025 109.86)
+		(width 1.27)
+		(layer "F.Cu")
+		(net "/V_out")
+	)
+	(segment
+		(start 72.2025 109.76)
+		(end 72.2025 104.5875)
+		(width 1.27)
+		(layer "F.Cu")
+		(net "/V_out")
+	)
+	(segment
+		(start 80.69 90.41)
+		(end 83.01 92.73)
+		(width 0.3)
+		(layer "F.Cu")
+		(net "/V_out")
+	)
+	(segment
+		(start 77.57 90.41)
+		(end 80.69 90.41)
+		(width 0.3)
+		(layer "F.Cu")
+		(net "/V_out")
+	)
+	(segment
+		(start 91.35 108.64)
+		(end 91.35 101.56)
+		(width 1.27)
+		(layer "F.Cu")
+		(net "/V_out")
+	)
+	(segment
+		(start 91.35 101.56)
+		(end 91.33 101.54)
+		(width 1.27)
+		(layer "F.Cu")
+		(net "/V_out")
+	)
+	(segment
+		(start 83.01 92.73)
+		(end 83.01 95.27)
+		(width 0.3)
+		(layer "F.Cu")
+		(net "/V_out")
+	)
+	(segment
+		(start 72.1025 109.86)
+		(end 72.2025 109.76)
+		(width 1.27)
+		(layer "F.Cu")
+		(net "/V_out")
+	)
+	(segment
+		(start 72.21 104.58)
+		(end 72.2025 104.5875)
+		(width 1.27)
+		(layer "F.Cu")
+		(net "/V_out")
+	)
+	(segment
+		(start 72.1525 100.5375)
+		(end 72.52 100.17)
+		(width 0.508)
+		(layer "F.Cu")
+		(net "/V_out")
+	)
+	(segment
 		(start 105.775 36.51)
 		(end 105.775 36.195)
@@
 	)
 	(segment
-		(start 67.65 109.86)
-		(end 72.1025 109.86)
-		(width 1.27)
-		(layer "F.Cu")
-		(net "/V_out")
-	)
-	(segment
-		(start 72.2025 109.76)
-		(end 72.2025 104.5875)
-		(width 1.27)
-		(layer "F.Cu")
-		(net "/V_out")
-	)
-	(segment
-		(start 80.69 90.41)
-		(end 83.01 92.73)
-		(width 0.3)
-		(layer "F.Cu")
-		(net "/V_out")
-	)
-	(segment
-		(start 77.57 90.41)
-		(end 80.69 90.41)
-		(width 0.3)
-		(layer "F.Cu")
-		(net "/V_out")
-	)
-	(segment
-		(start 91.35 108.64)
-		(end 91.35 101.56)
-		(width 1.27)
-		(layer "F.Cu")
-		(net "/V_out")
-	)
-	(segment
-		(start 91.35 101.56)
-		(end 91.33 101.54)
-		(width 1.27)
-		(layer "F.Cu")
-		(net "/V_out")
-	)
-	(segment
-		(start 83.01 92.73)
-		(end 83.01 95.27)
-		(width 0.3)
-		(layer "F.Cu")
-		(net "/V_out")
-	)
-	(segment
-		(start 72.1025 109.86)
-		(end 72.2025 109.76)
-		(width 1.27)
-		(layer "F.Cu")
-		(net "/V_out")
-	)
-	(segment
-		(start 72.21 104.58)
-		(end 72.2025 104.5875)
-		(width 1.27)
-		(layer "F.Cu")
-		(net "/V_out")
-	)
-	(segment
-		(start 72.1525 100.5375)
-		(end 72.52 100.17)
-		(width 0.508)
-		(layer "F.Cu")
-		(net "/V_out")
-	)
-	(segment
 		(start 48.59 108.69)
 		(end 48.59 102.01)
@@
 	)
 	(segment
-		(start 35.63 77.2)
-		(end 32.73 74.3)
+		(start 86.39 89.06)
+		(end 86.38 89.05)
 		(width 0.508)
 		(layer "B.Cu")
@@
 	)
 	(segment
-		(start 86.39 89.06)
-		(end 86.38 89.05)
+		(start 58.45 89.05)
+		(end 46.6 77.2)
 		(width 0.508)
 		(layer "B.Cu")
@@
 	)
 	(segment
-		(start 32.73 74.3)
-		(end 32.73 73.62)
+		(start 46.6 77.2)
+		(end 35.63 77.2)
 		(width 0.508)
 		(layer "B.Cu")
@@
 	)
 	(segment
-		(start 58.45 89.05)
-		(end 46.6 77.2)
+		(start 86.49 89.06)
+		(end 86.39 89.06)
 		(width 0.508)
 		(layer "B.Cu")
@@
 	)
 	(segment
-		(start 86.49 89.06)
-		(end 86.39 89.06)
+		(start 35.63 77.2)
+		(end 32.73 74.3)
 		(width 0.508)
 		(layer "B.Cu")
@@
 	)
 	(segment
-		(start 46.6 77.2)
-		(end 35.63 77.2)
+		(start 32.73 74.3)
+		(end 32.73 73.62)
 		(width 0.508)
 		(layer "B.Cu")
@@
 		(polygon
 			(pts
-				(xy 34.176817 97.486) (xy 35.38815 96.048103) (xy 39.095435 96.052363) (xy 40.584336 97.289295)
-				(xy 41.79 99.29) (xy 43.289032 99.3) (xy 43.69 99.71) (xy 43.69 100.96) (xy 41.14 103.33) (xy 40.24 103.56)
-				(xy 39.07 103.76) (xy 34.96 103.75) (xy 34.205917 102.704567)
+				(xy 34.174536 97.076913) (xy 35.041575 96.047705) (xy 39.095435 96.052363) (xy 40.654293 97.347413)
+				(xy 41.64751 98.99558) (xy 43.000143 99.004603) (xy 43.69 99.71) (xy 43.69 100.96) (xy 41.14 103.33)
+				(xy 40.24 103.56) (xy 39.07 103.76) (xy 34.96 103.75) (xy 34.205917 102.704567)
 			)
 		)
@@
 			(pts
 				(xy 37.173884 84.465461) (xy 38.262352 84.539953) (xy 39.51008 84.663172) (xy 45.477761 85.778294)
-				(xy 49.313884 86.785461) (xy 52.373884 89.415461) (xy 52.134156 98.725321) (xy 50.807892 100.252316)
+				(xy 46.883357 86.147331) (xy 51.641787 90.237092) (xy 51.420333 98.837293) (xy 50.204039 100.237673)
 				(xy 44.858332 100.108048) (xy 44.159578 99.588271) (xy 44.032933 98.72603) (xy 45.693884 94.355461)
 				(xy 45.324042 91.115641) (xy 37.116598 87.90461) (xy 36.893884 87.692336) (xy 36.913884 84.575461)
@@
 			(pts
 				(xy 32.73 88.63) (xy 32.97 88.01) (xy 32.97 83.39) (xy 34.457858 82.479067) (xy 35.69 82.17) (xy 36.386012 81.228337)
-				(xy 36.033418 79.629074) (xy 33.96165 78.523377) (xy 30.007608 80.053043) (xy 27.993321 83.132908)
-				(xy 28.126905 88.075477) (xy 28.82 88.87)
+				(xy 36.033418 79.629074) (xy 33.96165 78.523377) (xy 30.007608 80.053043) (xy 28.407814 82.499144)
+				(xy 28.552429 87.84986) (xy 29.410712 88.833741)
 			)
 		)
@@
 		(polygon
 			(pts
-				(xy 35.973861 83.201587) (xy 34.239391 83.037775) (xy 33.1 83.84) (xy 33.17 88.062504) (xy 32.72 88.73)
-				(xy 30.11 90.04) (xy 28.343576 93.527425) (xy 27.95 99.98) (xy 28.789598 100.72197) (xy 33.253682 100.637969)
-				(xy 33.63 100.11) (xy 34 95.01) (xy 35.47 91.45) (xy 36.52 86.9) (xy 36.383494 84.430486)
+				(xy 35.973861 83.201587) (xy 34.239391 83.037775) (xy 33.196381 83.77214) (xy 33.263662 87.830572)
+				(xy 32.495623 88.969823) (xy 30.023605 90.210568) (xy 28.981825 92.26734) (xy 28.758056 98.796127)
+				(xy 29.45 99.39) (xy 32.75 99.26) (xy 33.622868 98.184727) (xy 34.242488 94.422749) (xy 35.47 91.45)
+				(xy 36.52 86.9) (xy 36.383494 84.430486)
 			)
 		)

Commit message: Dioda
Parts:
- turned D13 to 0 degrees
Connections:
- D13 pad 1: Net-(D13-K) -> +5V
- D13 pad 2: +5V -> Net-(D13-A)
- J7 pad A4: Net-(D13-K) -> Net-(D13-A)
- J7 pad A9: Net-(D13-K) -> Net-(D13-A)
- J7 pad B4: Net-(D13-K) -> Net-(D13-A)
- J7 pad B9: Net-(D13-K) -> Net-(D13-A)
Routing:
- net Net-(D13-K): track 14.7 -> 0.00 mm
- net Net-(D13-A): track 0.00 -> 14.7 mm
Changed lines of the file:
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@@
 			(layers "F.Cu" "F.Mask" "F.Paste")
 			(roundrect_rratio 0.25)
-			(net "Net-(D13-K)")
+			(net "Net-(D13-A)")
 			(pinfunction "VBUS_A4")
 			(pintype "passive")
@@
 			(layers "F.Cu" "F.Mask" "F.Paste")
 			(roundrect_rratio 0.25)
-			(net "Net-(D13-K)")
+			(net "Net-(D13-A)")
 			(pinfunction "VBUS_A9")
 			(pintype "passive")
@@
 			(layers "F.Cu" "F.Mask" "F.Paste")
 			(roundrect_rratio 0.25)
-			(net "Net-(D13-K)")
+			(net "Net-(D13-A)")
 			(pinfunction "VBUS_B4")
 			(pintype "passive")
@@
 			(layers "F.Cu" "F.Mask" "F.Paste")
 			(roundrect_rratio 0.25)
-			(net "Net-(D13-K)")
+			(net "Net-(D13-A)")
 			(pinfunction "VBUS_B9")
 			(pintype "passive")
@@
 	(footprint "Diode_SMD:D_SMB_Handsoldering"
 		(layer "F.Cu")
-		(at 99.8 31.04 180)
+		(at 99.8 31.04)
 		(descr "Diode SMB (DO-214AA) Handsoldering")
 		(tags "Diode SMB (DO-214AA) Handsoldering")
@@
 		)
 		(property "Datasheet" "https://www.vishay.com/docs/88751/ss32.pdf"
-			(at 0 0 180)
+			(at 0 0 0)
 			(unlocked yes)
 			(layer "F.Fab")
@@
 		)
 		(property "Description" "40V 3A Schottky Diode, SMA"
-			(at 0 0 180)
+			(at 0 0 0)
 			(unlocked yes)
 			(layer "F.Fab")
@@
 		(duplicate_pad_numbers_are_jumpers no)
 		(fp_line
-			(start -4.71 2.15)
-			(end 2.7 2.15)
+			(start -4.71 -2.15)
+			(end -4.71 2.15)
 			(stroke
 				(width 0.12)
@@
 		)
 		(fp_line
-			(start -4.71 -2.15)
-			(end -4.71 2.15)
+			(start -4.71 2.15)
+			(end 2.7 2.15)
 			(stroke
 				(width 0.12)
@@
 		)
 		(fp_line
-			(start 4.7 2.25)
-			(end -4.7 2.25)
+			(start -4.7 -2.25)
+			(end 4.7 -2.25)
 			(stroke
 				(width 0.05)
@@
 		)
 		(fp_line
-			(start 4.7 -2.25)
-			(end 4.7 2.25)
+			(start -4.7 2.25)
+			(end -4.7 -2.25)
 			(stroke
 				(width 0.05)
@@
 		)
 		(fp_line
-			(start -4.7 2.25)
-			(end -4.7 -2.25)
+			(start 4.7 -2.25)
+			(end 4.7 2.25)
 			(stroke
 				(width 0.05)
@@
 		)
 		(fp_line
-			(start -4.7 -2.25)
-			(end 4.7 -2.25)
+			(start 4.7 2.25)
+			(end -4.7 2.25)
 			(stroke
 				(width 0.05)
@@
 		)
 		(fp_line
-			(start 2.3 2)
-			(end -2.3 2)
+			(start -2.3 2)
+			(end -2.3 -2)
 			(stroke
 				(width 0.1)
@@
 		)
 		(fp_line
-			(start 2.3 -2)
-			(end 2.3 2)
+			(start -0.64944 -0.79908)
+			(end -0.64944 0.80112)
 			(stroke
 				(width 0.1)
@@
 		)
 		(fp_line
-			(start 2.3 -2)
-			(end -2.3 -2)
+			(start -0.64944 0.00102)
+			(end -1.55114 0.00102)
 			(stroke
 				(width 0.1)
@@
 		)
 		(fp_line
-			(start 0.50118 0.75032)
+			(start -0.64944 0.00102)
 			(end 0.50118 -0.79908)
 			(stroke
@@
 		)
 		(fp_line
-			(start 0.50118 0.00102)
-			(end 1.4994 0.00102)
+			(start -0.64944 0.00102)
+			(end 0.50118 0.75032)
 			(stroke
 				(width 0.1)
@@
 		)
 		(fp_line
-			(start -0.64944 0.00102)
-			(end 0.50118 0.75032)
+			(start 0.50118 0.00102)
+			(end 1.4994 0.00102)
 			(stroke
 				(width 0.1)
@@
 		)
 		(fp_line
-			(start -0.64944 0.00102)
+			(start 0.50118 0.75032)
 			(end 0.50118 -0.79908)
 			(stroke
@@
 		)
 		(fp_line
-			(start -0.64944 0.00102)
-			(end -1.55114 0.00102)
+			(start 2.3 -2)
+			(end -2.3 -2)
 			(stroke
 				(width 0.1)
@@
 		)
 		(fp_line
-			(start -0.64944 -0.79908)
-			(end -0.64944 0.80112)
+			(start 2.3 -2)
+			(end 2.3 2)
 			(stroke
 				(width 0.1)
@@
 		)
 		(fp_line
-			(start -2.3 2)
-			(end -2.3 -2)
+			(start 2.3 2)
+			(end -2.3 2)
 			(stroke
 				(width 0.1)
@@
 		)
 		(pad "1" smd roundrect
-			(at -2.7 0 180)
+			(at -2.7 0)
 			(size 3.5 2.3)
 			(layers "F.Cu" "F.Mask" "F.Paste")
 			(roundrect_rratio 0.1086956522)
-			(net "Net-(D13-K)")
+			(net "+5V")
 			(pinfunction "K_1")
 			(pintype "passive")
 		)
 		(pad "2" smd roundrect
-			(at 2.7 0 180)
+			(at 2.7 0)
 			(size 3.5 2.3)
 			(layers "F.Cu" "F.Mask" "F.Paste")
 			(roundrect_rratio 0.1086956522)
-			(net "+5V")
+			(net "Net-(D13-A)")
 			(pinfunction "A_2")
 			(pintype "passive")
@@
 	)
 	(segment
-		(start 107.14 39.523604)
-		(end 107.14 38.135305)
-		(width 0.3)
-		(layer "F.Cu")
-		(net "Net-(D13-K)")
-	)
-	(segment
-		(start 106.314695 37.31)
-		(end 105.775 37.31)
-		(width 0.3)
-		(layer "F.Cu")
-		(net "Net-(D13-K)")
-	)
-	(segment
-		(start 102.5 34.87)
-		(end 104.94 37.31)
-		(width 0.508)
-		(layer "F.Cu")
-		(net "Net-(D13-K)")
-	)
-	(segment
-		(start 105.775 42.11)
-		(end 106.314695 42.11)
-		(width 0.3)
-		(layer "F.Cu")
-		(net "Net-(D13-K)")
-	)
-	(segment
-		(start 107.14 40.446396)
-		(end 107.15 40.436396)
-		(width 0.3)
-		(layer "F.Cu")
-		(net "Net-(D13-K)")
-	)
-	(segment
-		(start 102.5 31.04)
-		(end 102.5 34.87)
-		(width 0.508)
-		(layer "F.Cu")
-		(net "Net-(D13-K)")
-	)
-	(segment
-		(start 107.15 39.533604)
-		(end 107.14 39.523604)
-		(width 0.3)
-		(layer "F.Cu")
-		(net "Net-(D13-K)")
-	)
-	(segment
-		(start 106.314695 42.11)
-		(end 107.14 41.284695)
-		(width 0.3)
-		(layer "F.Cu")
-		(net "Net-(D13-K)")
-	)
-	(segment
-		(start 107.14 41.284695)
-		(end 107.14 40.446396)
-		(width 0.3)
-		(layer "F.Cu")
-		(net "Net-(D13-K)")
-	)
-	(segment
-		(start 104.94 37.31)
-		(end 105.775 37.31)
-		(width 0.508)
-		(layer "F.Cu")
-		(net "Net-(D13-K)")
-	)
-	(segment
-		(start 107.14 38.135305)
-		(end 106.314695 37.31)
-		(width 0.3)
-		(layer "F.Cu")
-		(net "Net-(D13-K)")
-	)
-	(segment
-		(start 107.15 40.436396)
-		(end 107.15 39.533604)
-		(width 0.3)
-		(layer "F.Cu")
-		(net "Net-(D13-K)")
-	)
-	(segment
 		(start 105.775 40.96)
 		(end 104.56 40.96)
@@
 		(net "Net-(Q2-G)")
 	)
+	(segment
+		(start 107.14 39.523604)
+		(end 107.14 38.135305)
+		(width 0.3)
+		(layer "F.Cu")
+		(net "Net-(D13-A)")
+	)
+	(segment
+		(start 106.314695 37.31)
+		(end 105.775 37.31)
+		(width 0.3)
+		(layer "F.Cu")
+		(net "Net-(D13-A)")
+	)
+	(segment
+		(start 102.5 34.87)
+		(end 104.94 37.31)
+		(width 0.508)
+		(layer "F.Cu")
+		(net "Net-(D13-A)")
+	)
+	(segment
+		(start 105.775 42.11)
+		(end 106.314695 42.11)
+		(width 0.3)
+		(layer "F.Cu")
+		(net "Net-(D13-A)")
+	)
+	(segment
+		(start 107.14 40.446396)
+		(end 107.15 40.436396)
+		(width 0.3)
+		(layer "F.Cu")
+		(net "Net-(D13-A)")
+	)
+	(segment
+		(start 102.5 31.04)
+		(end 102.5 34.87)
+		(width 0.508)
+		(layer "F.Cu")
+		(net "Net-(D13-A)")
+	)
+	(segment
+		(start 107.15 39.533604)
+		(end 107.14 39.523604)
+		(width 0.3)
+		(layer "F.Cu")
+		(net "Net-(D13-A)")
+	)
+	(segment
+		(start 106.314695 42.11)
+		(end 107.14 41.284695)
+		(width 0.3)
+		(layer "F.Cu")
+		(net "Net-(D13-A)")
+	)
+	(segment
+		(start 107.14 41.284695)
+		(end 107.14 40.446396)
+		(width 0.3)
+		(layer "F.Cu")
+		(net "Net-(D13-A)")
+	)
+	(segment
+		(start 104.94 37.31)
+		(end 105.775 37.31)
+		(width 0.508)
+		(layer "F.Cu")
+		(net "Net-(D13-A)")
+	)
+	(segment
+		(start 107.14 38.135305)
+		(end 106.314695 37.31)
+		(width 0.3)
+		(layer "F.Cu")
+		(net "Net-(D13-A)")
+	)
+	(segment
+		(start 107.15 40.436396)
+		(end 107.15 39.533604)
+		(width 0.3)
+		(layer "F.Cu")
+		(net "Net-(D13-A)")
+	)
 	(zone
