File: BMS.kicad_pcb (KiCad board)
At the start: 4 copper layers, 86 x 86 mm, 119 parts, among them J1 Conn_01x06_Pin, J2 Conn_01x02_Pin, J5 Conn_01x02_Pin, J6 Conn_01x04_Pin, J7 USB_C_Receptacle_USB2.0_16P, Q1 MMFTP3401-AQ, Q2 2N7002, Q3 SS8050, Q4 IRLZ44N, Q5 IRLZ44N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

Commit message: KOndensator
Parts:
- added C14: 100n, Capacitor_SMD:C_0805_2012Metric_Pad1.18x1.45mm_HandSolder, B.Cu at (91.7, 37.2)
- moved R9 0.15 mm to (94.6, 40.6)
Routing:
- net +5V: track 171.0 -> 172.7 mm
Changed lines of the file:
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@@
 	(footprint "Resistor_SMD:R_0805_2012Metric_Pad1.20x1.40mm_HandSolder"
 		(layer "B.Cu")
-		(at 94.75 40.62 -90)
+		(at 94.6 40.61 -90)
 		(descr "Resistor SMD 0805 (2012 Metric), square (rectangular) end terminal, IPC-7351 nominal with elongated pad for handsoldering. (Body size source: IPC-SM-782 page 72, https://www.pcb-3d.com/wordpress/wp-content/uploads/ipc-sm-782a_amendment_1_and_2.pdf)")
 		(tags "resistor handsolder")
@@
 		)
 	)
+	(footprint "Capacitor_SMD:C_0805_2012Metric_Pad1.18x1.45mm_HandSolder"
+		(layer "B.Cu")
+		(at 91.735 37.245 180)
+		(descr "Capacitor SMD 0805 (2012 Metric), square (rectangular) end terminal, IPC-7351 nominal with elongated pad for handsoldering. (Body size source: IPC-SM-782 page 76, https://www.pcb-3d.com/wordpress/wp-content/uploads/ipc-sm-782a_amendment_1_and_2.pdf, https://docs.google.com/spreadsheets/d/1BsfQQcO9C6DZCsRaXUlFlo91Tg2WpOkGARC1WS5S8t0/edit?usp=sharing)")
+		(tags "capacitor handsolder")
+		(property "Reference" "C14"
+			(at 0 1.68 0)
+			(layer "B.SilkS")
+			(effects
+				(font
+					(size 1 1)
+					(thickness 0.15)
+				)
+				(justify mirror)
+			)
+		)
+		(property "Value" "100n"
+			(at 0 -1.68 0)
+			(layer "B.Fab")
+			(effects
+				(font
+					(size 1 1)
+					(thickness 0.15)
+				)
+				(justify mirror)
+			)
+		)
+		(property "Datasheet" ""
+			(at 0 0 0)
+			(layer "B.Fab")
+			(hide yes)
+			(effects
+				(font
+					(size 1.27 1.27)
+				)
+				(justify mirror)
+			)
+		)
+		(property "Description" "Unpolarized capacitor"
+			(at 0 0 0)
+			(layer "B.Fab")
+			(hide yes)
+			(effects
+				(font
+					(size 1.27 1.27)
+				)
+				(justify mirror)
+			)
+		)
+		(property ki_fp_filters "C_*")
+		(sheetname "/")
+		(sheetfile "BMS.kicad_sch")
+		(units
+			(unit
+				(name "A")
+				(pins "1" "2")
+			)
+		)
+		(attr smd)
+		(duplicate_pad_numbers_are_jumpers no)
+		(fp_line
+			(start -0.261252 0.735)
+			(end 0.261252 0.735)
+			(stroke
+				(width 0.12)
+				(type solid)
+			)
+			(layer "B.SilkS")
+		)
+		(fp_line
+			(start -0.261252 -0.735)
+			(end 0.261252 -0.735)
+			(stroke
+				(width 0.12)
+				(type solid)
+			)
+			(layer "B.SilkS")
+		)
+		(fp_rect
+			(start -1.88 0.98)
+			(end 1.88 -0.98)
+			(stroke
+				(width 0.05)
+				(type solid)
+			)
+			(fill no)
+			(layer "B.CrtYd")
+		)
+		(fp_rect
+			(start -1 0.625)
+			(end 1 -0.625)
+			(stroke
+				(width 0.1)
+				(type solid)
+			)
+			(fill no)
+			(layer "B.Fab")
+		)
+		(fp_text user "${REFERENCE}"
+			(at 0 0 0)
+			(layer "B.Fab")
+			(effects
+				(font
+					(size 0.5 0.5)
+					(thickness 0.08)
+				)
+				(justify mirror)
+			)
+		)
+		(pad "1" smd roundrect
+			(at -1.0375 0 180)
+			(size 1.175 1.45)
+			(layers "B.Cu" "B.Mask" "B.Paste")
+			(roundrect_rratio 0.212766)
+			(net "+5V")
+			(pintype "passive")
+		)
+		(pad "2" smd roundrect
+			(at 1.0375 0 180)
+			(size 1.175 1.45)
+			(layers "B.Cu" "B.Mask" "B.Paste")
+			(roundrect_rratio 0.212766)
+			(net "GND")
+			(pintype "passive")
+		)
+		(embedded_fonts no)
+		(model "${KICAD10_3DMODEL_DIR}/Capacitor_SMD.3dshapes/C_0805_2012Metric.step"
+			(offset
+				(xyz 0 0 0)
+			)
+			(scale
+				(xyz 1 1 1)
+			)
+			(rotate
+				(xyz 0 0 0)
+			)
+		)
+	)
 	(footprint "Resistor_SMD:R_0805_2012Metric_Pad1.20x1.40mm_HandSolder"
 		(layer "B.Cu")
@@
 	)
 	(segment
-		(start 94.593176 37.281226)
-		(end 94.75 37.43805)
+		(start 94.6 39.47)
+		(end 94.6 39.61)
 		(width 0.3)
 		(layer "B.Cu")
@@
 	)
 	(segment
-		(start 94.75 37.43805)
-		(end 94.75 39.62)
-		(width 0.3)
+		(start 89.27 78.8175)
+		(end 87.1675 78.8175)
+		(width 1.1)
 		(layer "B.Cu")
 		(net "+5V")
 	)
 	(segment
-		(start 89.27 78.8175)
-		(end 87.1675 78.8175)
-		(width 1.1)
+		(start 94.593176 37.266824)
+		(end 94.593176 39.463176)
+		(width 0.3)
 		(layer "B.Cu")
 		(net "+5V")
@@
 	)
 	(segment
-		(start 89.27 78.8175)
-		(end 93.5275 78.8175)
-		(width 1.1)
+		(start 92.794324 37.266824)
+		(end 92.7725 37.245)
+		(width 0.3)
+		(layer "B.Cu")
+		(net "+5V")
+	)
+	(segment
+		(start 94.593176 39.463176)
+		(end 94.6 39.47)
+		(width 0.3)
 		(layer "B.Cu")
 		(net "+5V")
@@
 	(segment
 		(start 94.593176 37.266824)
-		(end 94.593176 37.281226)
+		(end 92.794324 37.266824)
 		(width 0.3)
 		(layer "B.Cu")
@@
 	)
 	(segment
+		(start 89.27 78.8175)
+		(end 93.5275 78.8175)
+		(width 1.1)
+		(layer "B.Cu")
+		(net "+5V")
+	)
+	(segment
 		(start 44.77 83.96)
 		(end 44.93 84.12)
@@
 	)
 	(segment
+		(start 107.14 39.523604)
+		(end 107.14 38.135305)
+		(width 0.3)
+		(layer "F.Cu")
+		(net "Net-(D13-A)")
+	)
+	(segment
+		(start 106.314695 37.31)
+		(end 105.775 37.31)
+		(width 0.3)
+		(layer "F.Cu")
+		(net "Net-(D13-A)")
+	)
+	(segment
+		(start 102.5 34.87)
+		(end 104.94 37.31)
+		(width 0.508)
+		(layer "F.Cu")
+		(net "Net-(D13-A)")
+	)
+	(segment
+		(start 105.775 42.11)
+		(end 106.314695 42.11)
+		(width 0.3)
+		(layer "F.Cu")
+		(net "Net-(D13-A)")
+	)
+	(segment
+		(start 107.14 40.446396)
+		(end 107.15 40.436396)
+		(width 0.3)
+		(layer "F.Cu")
+		(net "Net-(D13-A)")
+	)
+	(segment
+		(start 102.5 31.04)
+		(end 102.5 34.87)
+		(width 0.508)
+		(layer "F.Cu")
+		(net "Net-(D13-A)")
+	)
+	(segment
+		(start 107.15 39.533604)
+		(end 107.14 39.523604)
+		(width 0.3)
+		(layer "F.Cu")
+		(net "Net-(D13-A)")
+	)
+	(segment
+		(start 106.314695 42.11)
+		(end 107.14 41.284695)
+		(width 0.3)
+		(layer "F.Cu")
+		(net "Net-(D13-A)")
+	)
+	(segment
+		(start 107.14 41.284695)
+		(end 107.14 40.446396)
+		(width 0.3)
+		(layer "F.Cu")
+		(net "Net-(D13-A)")
+	)
+	(segment
+		(start 104.94 37.31)
+		(end 105.775 37.31)
+		(width 0.508)
+		(layer "F.Cu")
+		(net "Net-(D13-A)")
+	)
+	(segment
+		(start 107.14 38.135305)
+		(end 106.314695 37.31)
+		(width 0.3)
+		(layer "F.Cu")
+		(net "Net-(D13-A)")
+	)
+	(segment
+		(start 107.15 40.436396)
+		(end 107.15 39.533604)
+		(width 0.3)
+		(layer "F.Cu")
+		(net "Net-(D13-A)")
+	)
+	(segment
 		(start 105.775 40.96)
 		(end 104.56 40.96)
@@
 	)
 	(segment
-		(start 94.9625 43.5625)
-		(end 96.44 43.5625)
+		(start 94.73 43.05)
+		(end 94.73 43.33)
 		(width 0.3)
 		(layer "F.Cu")
@@
 	)
 	(segment
-		(start 94.73 43.33)
-		(end 94.9625 43.5625)
+		(start 94.9625 43.5625)
+		(end 96.44 43.5625)
 		(width 0.3)
 		(layer "F.Cu")
@@
 	)
 	(segment
-		(start 94.73 43.05)
-		(end 94.73 43.33)
+		(start 94.73 43.33)
+		(end 94.9625 43.5625)
 		(width 0.3)
 		(layer "F.Cu")
@@
 	)
 	(segment
-		(start 94.73 41.77)
-		(end 94.75 41.75)
+		(start 94.73 43.05)
+		(end 94.7 43.02)
 		(width 0.3)
 		(layer "B.Cu")
@@
 	)
 	(segment
-		(start 94.73 43.05)
-		(end 94.73 41.77)
+		(start 94.7 43.02)
+		(end 94.7 41.71)
 		(width 0.3)
 		(layer "B.Cu")
@@
 	)
 	(segment
-		(start 94.75 41.75)
-		(end 94.75 41.62)
+		(start 94.7 41.71)
+		(end 94.6 41.61)
 		(width 0.3)
 		(layer "B.Cu")
@@
 		(net "Net-(Q2-G)")
 	)
-	(segment
-		(start 107.14 39.523604)
-		(end 107.14 38.135305)
-		(width 0.3)
-		(layer "F.Cu")
-		(net "Net-(D13-A)")
-	)
-	(segment
-		(start 106.314695 37.31)
-		(end 105.775 37.31)
-		(width 0.3)
-		(layer "F.Cu")
-		(net "Net-(D13-A)")
-	)
-	(segment
-		(start 102.5 34.87)
-		(end 104.94 37.31)
-		(width 0.508)
-		(layer "F.Cu")
-		(net "Net-(D13-A)")
-	)
-	(segment
-		(start 105.775 42.11)
-		(end 106.314695 42.11)
-		(width 0.3)
-		(layer "F.Cu")
-		(net "Net-(D13-A)")
-	)
-	(segment
-		(start 107.14 40.446396)
-		(end 107.15 40.436396)
-		(width 0.3)
-		(layer "F.Cu")
-		(net "Net-(D13-A)")
-	)
-	(segment
-		(start 102.5 31.04)
-		(end 102.5 34.87)
-		(width 0.508)
-		(layer "F.Cu")
-		(net "Net-(D13-A)")
-	)
-	(segment
-		(start 107.15 39.533604)
-		(end 107.14 39.523604)
-		(width 0.3)
-		(layer "F.Cu")
-		(net "Net-(D13-A)")
-	)
-	(segment
-		(start 106.314695 42.11)
-		(end 107.14 41.284695)
-		(width 0.3)
-		(layer "F.Cu")
-		(net "Net-(D13-A)")
-	)
-	(segment
-		(start 107.14 41.284695)
-		(end 107.14 40.446396)
-		(width 0.3)
-		(layer "F.Cu")
-		(net "Net-(D13-A)")
-	)
-	(segment
-		(start 104.94 37.31)
-		(end 105.775 37.31)
-		(width 0.508)
-		(layer "F.Cu")
-		(net "Net-(D13-A)")
-	)
-	(segment
-		(start 107.14 38.135305)
-		(end 106.314695 37.31)
-		(width 0.3)
-		(layer "F.Cu")
-		(net "Net-(D13-A)")
-	)
-	(segment
-		(start 107.15 40.436396)
-		(end 107.15 39.533604)
-		(width 0.3)
-		(layer "F.Cu")
-		(net "Net-(D13-A)")
-	)
 	(zone

Commit message: rezystor V_out
Parts:
- removed R27: 1k, Resistor_SMD:R_0805_2012Metric_Pad1.20x1.40mm_HandSolder
- R47, R48: moved to F.Cu
- moved R48 5.17 mm to (65.7, 90.8), turned to 0 degrees
- moved R47 4.27 mm to (72.5, 90.9), turned to 180 degrees
- moved C3 1.77 mm to (49.7, 99.0), turned to 0 degrees
- moved D10 0.68 mm to (44.8, 93.1)
- moved Q1 0.35 mm to (43.5, 99.0)
- moved R3 0.13 mm to (37.6, 93.1)
- moved D11 0.12 mm to (31.2, 99.8)
Routing:
- net Net-(D10-K): track 0.00 -> 22.3 mm
- net Net-(D11-K): track 0.20 -> 14.1 mm
- net Net-(D10-A): track 0.00 -> 9.03 mm
- net +5V: track 172.7 -> 181.5 mm
- net +BATT: track 18.2 -> 23.1 mm
- net /V_out: track 26.3 -> 21.9 mm
- net Net-(Q8-G): track 2.81 -> 6.39 mm, vias 0 -> 1
- net Net-(R46-Pad1): track 12.5 -> 9.52 mm, vias 1 -> 0
- net Net-(Q7-G): track 3.90 -> 6.73 mm, vias 0 -> 1
- net Net-(R45-Pad1): track 12.5 -> 10.2 mm, vias 1 -> 0
- removed copper zone on B.Cu, net +5V
- removed copper zone on B.Cu, net +BATT
- removed copper zone on B.Cu, net Net-(D10-A)
- removed copper zone on B.Cu, net Net-(D10-K)
- removed copper zone on B.Cu, net Net-(D11-K)
