File: BMS.kicad_pcb (KiCad board)
At the start: 4 copper layers, 86 x 86 mm, 119 parts, among them J1 Conn_01x06_Pin, J2 Conn_01x02_Pin, J5 Conn_01x02_Pin, J6 Conn_01x04_Pin, J7 USB_C_Receptacle_USB2.0_16P, Q1 MMFTP3401-AQ, Q2 2N7002, Q3 SS8050, Q4 IRLZ44N, Q5 IRLZ44N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

Commit message: poprawiłem
Parts:
- removed C1: 100n, Capacitor_SMD:C_0805_2012Metric_Pad1.18x1.45mm_HandSolder
- removed C6, C9: 10u, Capacitor_SMD:C_0805_2012Metric_Pad1.18x1.45mm_HandSolder
- added C16: 100n, Capacitor_SMD:C_0805_2012Metric_Pad1.18x1.45mm_HandSolder, B.Cu at (42.3, 103.2)
- added C18: 100n, Capacitor_SMD:C_0805_2012Metric_Pad1.18x1.45mm_HandSolder, B.Cu at (32.2, 78.3)
- added C26: 10u, Capacitor_SMD:CP_Elec_5x4.5, B.Cu at (90.7, 85.0)
- added C27: 10u, Capacitor_SMD:CP_Elec_5x4.5, B.Cu at (98.7, 85.0)
- added C28: 100n, Capacitor_SMD:C_0603_1608Metric, F.Cu at (109.8, 60.0)
- added R27: 10k, Resistor_SMD:R_0805_2012Metric_Pad1.20x1.40mm_HandSolder, F.Cu at (110.7, 62.9)
- C2: value 22u -> 100n
- L1: footprint Inductor_SMD:L_7.3x7.3_H4.5 -> Inductor_SMD:L_Panasonic_PCC-M0630M
- moved R3 4.92 mm to (41.2, 89.7)
- moved L1 1.66 mm to (32.7, 91.4), turned to 180 degrees
- moved D11 0.34 mm to (31.0, 99.6)
Connections:
- U5 pad 4: unconnected-(U5-V3-Pad4) -> +3.3V
Routing:
- net +3.3V: track 137.2 -> 152.3 mm, vias 8 -> 9
- net +5V: track 181.5 -> 194.9 mm
- net Net-(C28-Pad1): track 20.3 -> 28.2 mm
- net /EN: track 69.3 -> 65.7 mm
- net GND: track 19.3 -> 15.8 mm, vias 213 -> 211
- net +BATT: track 23.1 -> 25.4 mm
- net Net-(D11-K): track 14.1 -> 15.7 mm
- net Net-(D10-A): track 9.03 -> 8.46 mm

Commit message: MILKA
Parts:
- added G***: LOGO, LOGO, F.Cu at (95.2, 68.5)
- added G***: LOGO, LOGO, B.Cu at (41.2, 46.1)
