File: Hardware/BMS.kicad_pcb (KiCad board)
At the start: 4 copper layers, 86 x 86 mm, 124 parts, among them J1 Conn_01x06_Pin, J2 Conn_01x02_Pin, J5 Conn_01x02_Pin, J6 Conn_01x04_Pin, J7 USB_C_Receptacle_USB2.0_16P, Q1 MMFTP3401-AQ, Q2 2N7002, Q3 SS8050, Q4 IRLZ44N, Q5 IRLZ44N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

Commit message: first commit
Parts:
- removed G*** (x2): LOGO, LOGO
